File: test_MP118FD.kicad_pcb (KiCad board)
At the start: 2 copper layers, 161 x 135.5 mm, 18 parts, among them J1 Screw_Terminal_01x01, J2 Screw_Terminal_01x01, J3 Conn_Coaxial

Commit message: Reconfiguración general, arreglos de redes y posiciones mas centradas
Parts:
- removed C7: 10 pF, Capacitor_THT:C_Disc_D7.5mm_W5.0mm_P7.50mm
- removed MP118DF1: MP118FD, Library:MP118
- removed TS1: Conn_01x07_Socket, Library:PhoenixContact_SPT_5_7-H-7.5-ZB_1x07_P7.5mm_Horizontal
- added Cc1: 10 pF, Capacitor_THT:C_Disc_D7.5mm_W5.0mm_P7.50mm, F.Cu at (158.7, 91.4)
- added J4: Conn_01x07_Socket, Library:PhoenixContact_SPT_5_7-H-7.5-ZB_1x07_P7.5mm_Horizontal, F.Cu at (206.1, 132.9)
- added U MP118DF1: ~, Library:MP118, F.Cu at (143.5, 85.1)
- R1: value 0.54 -> 1K; footprint Library:Shunt PBV Isabellenhutte 17,78x7,62 -> Resistor_THT:R_Axial_DIN0207_L6.3mm_D2.5mm_P7.62mm_Horizontal
- R2: value 1K -> 10K
- R4: value 10K -> 0.54; footprint Resistor_THT:R_Axial_DIN0207_L6.3mm_D2.5mm_P7.62mm_Horizontal -> Library:Shunt PBV Isabellenhutte 17,78x7,62
- moved R1 60.5 mm to (101.6, 137.2), turned to 90 degrees
- moved R4 47.7 mm to (166.3, 101.6)
- moved J2 32.2 mm to (91.4, 146.5)
- moved PB1 31.0 mm to (123.1, 58.4)
- moved C3 26.3 mm to (177.8, 147.2)
- moved J3 24.9 mm to (92.1, 121.3)
- moved C2 24.9 mm to (177.8, 65.9)
- moved C4 24.9 mm to (177.8, 111.8), turned to 0 degrees
- moved PB2 24.9 mm to (136.0, 53.4)
- moved C1 24.8 mm to (177.8, 91.4), turned to 0 degrees
- moved C6 22.1 mm to (144.8, 111.8), turned to 180 degrees
- moved C5 17.7 mm to (144.8, 91.4)
- moved R3 13.4 mm to (121.9, 134.6)
- moved J1 12.6 mm to (91.4, 137.2)
- moved R2 9.83 mm to (109.2, 134.6), turned to 0 degrees
Connections:
- C3 pad 1: /-Vb -> /-Vs
- C4 pad 1: /-Vb -> /-Vs
- R1 pad 1: Net-(MP118DF1-OUT-Pad13) -> Net-(U MP118DF1--IN)
- R1 pad 2: Net-(MP118DF1-+Isd) -> Net-(J1-Pin_1)
- R2 pad 1: Net-(MP118DF1--IN) -> Net-(U MP118DF1--IN)
- R2 pad 2: Net-(J1-Pin_1) -> Net-(R2-Pad2)
- R3 pad 1: Net-(MP118DF1--IN) -> Net-(R2-Pad2)
- R3 pad 2: Net-(R3-Pad2) -> /OUT
- R4 pad 1: Net-(R3-Pad2) -> Net-(R4-Pad1)
- R4 pad 2: /OUT -> Net-(U MP118DF1-+Isd)
Routing:
- removed copper zone on F.Cu, net (none)
Other:
- board size 161 x 135.5 mm -> 162.6 x 127 mm
- board text removed: "+Vb"
- board text removed: "+Vs"
- board text removed: "-Vb"
- board text removed: "-Vs"
- board text removed: "GND"
- board text removed: "OUT"
- board text removed: "SPARE"

Commit message: Hasta el viernes
Parts:
- added R5: 0, Resistor_THT:R_Axial_DIN0207_L6.3mm_D2.5mm_P7.62mm_Horizontal, F.Cu at (166.4, 124.5)
- moved C1 1.47 mm to (179.3, 91.5), turned to -90 degrees
- moved C4 1.46 mm to (179.3, 111.8), turned to 90 degrees
- moved J4 0.63 mm to (206.2, 132.3)
Connections:
- net Net-(R4-Pad1) renamed /OUT_0
- J4 pad 1: /-Vb -> /SPARE
- J4 pad 2: /-Vs -> /+Vs
- J4 pad 3: GND -> /+Vb
- J4 pad 5: /+Vb -> GND
- J4 pad 6: /+Vs -> /-Vs
- J4 pad 7: /SPARE -> /-Vb
Routing:
- net Net-(U MP118DF1-SD_): track 0.00 -> 56.1 mm
- net /+Vs: track 0.00 -> 51.5 mm
- net GND: track 0.00 -> 44.7 mm
- net Net-(PB2-A): track 0.00 -> 34.1 mm
- added copper zone on F.Cu, net /+Vs
- added copper zone on F.Cu, net /-Vs
